Commit message: rebasing

File: ik_ros_examples/configs/kuka_lwr_exotica_example/lwr.urdf (robot description, URDF)
Before this commit: robot lwr, 9 links, 8 joints
Links:
- removed link base
- added link base_link, mass 0.00000; collision box size=1 1 0.04; visual box size=1 1 0.04
Joints:
- joint base_joint: parent base -> base_link
